Commit message: Resolve YAM CAD provenance
Signed-off-by: Runyu Lu <runyul@nvidia.com>

File: aspire/real/robot/models/station/station_zed2itop.urdf (robot description, URDF)
Before this commit: robot station, 30 links, 29 joints
Links:
- link top_camera_zed2i: geometry visual box size=0.175232 0.030251 0.044102
